File: circut/pcb.kicad_pcb (KiCad board)
At the start: 2 copper layers, 22 x 71 mm, 17 parts, among them J1 GY-302, J2 LD2410B, J3 USB_C_Receptacle_USB2.0, Q1 S8050, U1 AMS1117-3.3, U2 HDC1080, U3 ESP32-S3-WROOM-1

Commit message: optimize pcb layout
Parts:
- added C4: 0.1uF, Capacitor_SMD:C_0805_2012Metric, F.Cu at (137.7, 151.4)
- D1: value IR204A -> IR
- U1: value AMS1117-3.3 -> AMS1117
- moved U2 43.8 mm to (137.7, 155.0)
- moved J2 35.5 mm to (155.8, 110.4), turned to -90 degrees
- moved R5 34.3 mm to (136.7, 147.8), turned to 90 degrees
- moved R4 32.3 mm to (138.7, 147.8), turned to 90 degrees
- moved U1 22.2 mm to (141.0, 121.0), turned to 180 degrees
- moved C1 21.6 mm to (147.3, 120.9), turned to 90 degrees
- moved J1 6.77 mm to (147.6, 127.3)
- moved R3 5.31 mm to (141.2, 109.3)
- moved D1 3.82 mm to (142.3, 112.5), turned to -90 degrees
- moved R1 2.24 mm to (137.4, 115.3)
- moved Q1 1.79 mm to (147.3, 114.3), turned to 90 degrees
- moved R2 1.65 mm to (148.0, 110.0)
- moved D2 1.05 mm to (145.0, 109.3), turned to 0 degrees
- moved C2 0.89 mm to (137.4, 112.3)
Connections:
- R2 pad 2: Net-(U3-GPIO12/TOUCH12/ADC2_CH1/FSPICLK/FSPIIO6/SUBSPICLK) -> Net-(U3-GPIO14/TOUCH14/ADC2_CH3/FSPIWP/FSPIDQS/SUBSPIWP)
- U3 pad 17: Net-(J1-Pin_3) -> unconnected-(U3-GPIO9/TOUCH9/ADC1_CH8/FSPIHD/SUBSPIHD-Pad17)
- U3 pad 18: Net-(J1-Pin_2) -> Net-(J1-Pin_3)
- U3 pad 19: Net-(D2-A) -> Net-(J1-Pin_2)
- U3 pad 20: Net-(U3-GPIO12/TOUCH12/ADC2_CH1/FSPICLK/FSPIIO6/SUBSPICLK) -> Net-(D2-A)
- U3 pad 21: Net-(J2-Pin_2) -> unconnected-(U3-GPIO13/TOUCH13/ADC2_CH2/FSPIQ/FSPIIO7/SUBSPIQ-Pad21)
- U3 pad 22: Net-(J2-Pin_3) -> Net-(U3-GPIO14/TOUCH14/ADC2_CH3/FSPIWP/FSPIDQS/SUBSPIWP)
- U3 pad 24: unconnected-(U3-GPIO47/SPICLK_P/SUBSPICLK_P_DIFF-Pad24) -> Net-(J2-Pin_3)
- U3 pad 25: unconnected-(U3-GPIO48/SPICLK_N/SUBSPICLK_N_DIFF-Pad25) -> Net-(J2-Pin_2)
Routing:
- net Net-(D1-A): track 74.5 -> 157.6 mm, vias 2 -> 0
- net Net-(J1-Pin_3): track 27.4 -> 110.5 mm, vias 2 -> 3
- net Net-(J1-Pin_2): track 25.5 -> 106.0 mm, vias 2 -> 3
- net Net-(J2-Pin_3): track 43.6 -> 5.48 mm
- net Net-(J2-Pin_2): track 43.3 -> 5.48 mm
- net /VCC: track 24.7 -> 61.0 mm
- net Net-(J1-Pin_4): track 161.5 -> 174.5 mm, vias 5 -> 14
- net Net-(U3-EN): track 35.0 -> 27.2 mm
- net Net-(J3-CC1): track 57.3 -> 64.4 mm
- net Net-(U3-GPIO12/TOUCH12/ADC2_CH1/FSPICLK/FSPIIO6/SUBSPICLK): track 5.86 -> 0.00 mm
- net Net-(U3-U0TXD/GPIO43/CLK_OUT1): track 67.1 -> 71.5 mm
- net Net-(U3-U0RXD/GPIO44/CLK_OUT2): track 65.9 -> 69.7 mm
- net Net-(U3-GPIO14/TOUCH14/ADC2_CH3/FSPIWP/FSPIDQS/SUBSPIWP): track 0.00 -> 2.93 mm
- net Net-(Q1-E): track 2.74 -> 5.30 mm
- net Net-(D1-K): track 3.81 -> 5.29 mm
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- added copper zone on B.Cu, net Net-(J1-Pin_4)
- added copper zone on F.Cu, net Net-(J1-Pin_4)
